Commit message: fix arm length and motor config

File: source/stabilization/stabilization/tasks/manager_based/stabilization/models/AerialManipulator_0dof.urdf (robot description, URDF)
Before this commit: robot Robot, 14 links, 13 joints
Links:
- link arm: mass None -> 1e-9
- link gripper: mass None -> 1e-9
- link motor1: mass None -> 1e-9
- link motor2: mass None -> 1e-9
- link motor3: mass None -> 1e-9
- link motor4: mass None -> 1e-9
- link prop1: mass None -> 1e-9
- link prop2: mass None -> 1e-9
- link prop3: mass None -> 1e-9
- link prop4: mass None -> 1e-9
- link quadrotor: mass None -> 1e-9
